File: schematic/5x5x2.kicad_pcb (KiCad board)
At the start: 2 copper layers, 100 x 100 mm, 158 parts, among them J1 SW Debug, J2 USB_C_Receptacle_USB2.0, SW1 SW, SW11 SW, SW12 SW, SW13 SW, SW14 SW, SW15 SW, SW21 SW, SW22 SW, SW23 SW, SW24 SW, SW25 SW, SW31 SW, SW32 SW, SW33 SW, SW34 SW, SW35 SW, SW41 SW, SW42 SW, SW43 SW, SW44 SW, SW45 SW, SW51 SW, SW52 SW, SW53 SW, SW54 SW, SW55 SW, SW6 ALPS_EC11, U1 SRV0504, U2 STM32F103C8, U3 LD1117S33CTR, Y1 16M

Commit message: Adjusted sk6812 footprint, started routing
Adjusted sk6812 footprint from square cutout to something that is
routable with a mill.

The kailh sockets and leds eat up all the space between the keys. This
means that there is not room for the micro, regulator and usb
receptacle if we stay in a 10x10.

Options:
- Increase size to 11x11 or even 12x12. This would allow for some nice
  mounting holes.

- Make another board beneath the switch board that contains the micro
  and friends.

Lets think about this some more.
Parts:
- added CB6: 100n, Capacitor_SMD:C_0805_2012Metric, F.Cu at (483.0, -134.5)
- added CB7: 100n, Capacitor_SMD:C_0805_2012Metric, F.Cu at (483.0, -137.5)
- added CB8: 100n, Capacitor_SMD:C_0805_2012Metric, F.Cu at (490.8, -143.2)
- added LEDB6: SK6812MINI, footprints:SK6812MINI_rev, F.Cu at (476.7, -136.2)
- added LEDB7: SK6812MINI, footprints:SK6812MINI_rev, F.Cu at (484.5, -141.8)
- added LEDB8: SK6812MINI, footprints:SK6812MINI_rev, F.Cu at (476.7, -141.8)
- C11, C12, C13, C14, C15, D31, D32, D33, D34, D35, D41, D42, D43, D44, D45, D51, D52, D53, D54, D55: moved to B.Cu
- moved C41 554.2 mm to (5.10, 82.0)
- moved C52 543.6 mm to (10.5, 89.5)
- moved C51 533.8 mm to (4.55, 89.5)
- moved C34 533.0 mm to (22.6, 74.5)
- moved C31 523.5 mm to (5.05, 74.0)
- moved C25 511.2 mm to (28.6, 67.0)
- moved C35 502.3 mm to (29.1, 74.5)
- moved C32 494.1 mm to (11.1, 74.5)
- moved C22 487.7 mm to (11.0, 67.5)
- moved C44 470.1 mm to (22.5, 82.5)
- moved C13 464.6 mm to (86.0, 59.5)
- moved C54 463.6 mm to (22.6, 89.5)
- moved U2 457.9 mm to (58.0, 37.0), turned to -45 degrees
- moved C23 455.4 mm to (17.1, 67.5)
- moved C55 446.7 mm to (28.1, 89.5)
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- renumbered C26 to C45
Connections:
- R15 pad 1: Net-(LEDB5-Pad2) -> GND
- R15 pad 2: GND -> Net-(LEDB8-Pad2)
Routing:
- net ROTD: track 0.00 -> 21.0 mm
- net Net-(LED11-Pad2): track 0.00 -> 14.1 mm
- net Net-(D11-Pad2): track 0.00 -> 4.00 mm

Commit message: More routing
Parts:
- C21, C22, C23, C24, C25, C31, C32, C33, C34, C35, C41, C42, C43, C44, C45, C51, C52, C53, C54, C55, CB5, LEDB1, LEDB2, LEDB3, LEDB4, LEDB5, LEDB6, LEDB7, LEDB8: moved to B.Cu
- moved LEDB4 460.9 mm to (37.5, 69.5), turned to -90 degrees
- moved LEDB3 443.2 mm to (37.5, 107.5), turned to -90 degrees
- moved LEDB2 438.3 mm to (67.2, 136.0), turned to 180 degrees
- moved CB1 430.8 mm to (73.0, 160.2)
- moved CB2 430.8 mm to (77.9, 160.2)
- moved CB3 430.8 mm to (83.5, 160.2)
- moved CB4 430.8 mm to (89.3, 160.2)
- moved LEDB8 423.7 mm to (133.8, 107.0), turned to -90 degrees
- moved CB5 414.6 mm to (100.2, 135.9), turned to -90 degrees
- moved LEDB6 411.7 mm to (104.8, 40.2), turned to 180 degrees
- moved LEDB7 409.2 mm to (133.8, 69.0), turned to -90 degrees
- moved LEDB5 401.5 mm to (66.5, 40.0), turned to 180 degrees
- moved LEDB1 397.6 mm to (105.0, 136.0)
- moved CB6 394.1 mm to (152.5, 80.3)
- moved CB7 394.1 mm to (152.5, 77.2)
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- renumbered LED25 to LED21, LED24 to LED22, LED22 to LED24, LED21 to LED25, LED45 to LED41, LED44 to LED42, LED42 to LED44, LED41 to LED45
Routing:
- net COL1: track 0.00 -> 94.6 mm, vias 0 -> 5
- net COL5: track 0.00 -> 86.6 mm, vias 0 -> 5
- net COL3: track 0.00 -> 85.6 mm, vias 0 -> 4
- net COL2: track 0.00 -> 85.6 mm, vias 0 -> 4
- net COL4: track 0.00 -> 85.5 mm, vias 0 -> 4
- net ROW2: track 0.00 -> 81.5 mm
- net ROW3: track 0.00 -> 81.5 mm
- net ROW5: track 0.00 -> 81.5 mm
- net ROW4: track 0.00 -> 81.5 mm
- net ROTD: track 21.0 -> 82.6 mm
- net Net-(LED41-Pad2): track 0.00 -> 28.0 mm
- net Net-(LED15-Pad2): track 0.00 -> 27.2 mm
- net Net-(LED21-Pad2): track 0.00 -> 27.1 mm
- net Net-(LED35-Pad2): track 0.00 -> 26.4 mm
- net ROTE: track 0.00 -> 23.0 mm
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
Commit message: Routed for mcu on other pcb
This way we can stay with 2 layers, and optionally have an additional
pcb for just the key switches without kailh holders.
Parts:
- added REF**: MountingHole_3.2mm_M3, MountingHole:MountingHole_3.2mm_M3, F.Cu at (39.5, 41.5)
- added REF**: PinSocket_1x05_P2.54mm_Vertical, Connector_PinSocket_2.54mm:PinSocket_1x05_P2.54mm_Vertical, B.Cu at (52.5, 116.5)
- added REF**: MountingHole_3.2mm_M3, MountingHole:MountingHole_3.2mm_M3, F.Cu at (39.5, 134.5)
- added REF**: MountingHole_3.2mm_M3, MountingHole:MountingHole_3.2mm_M3, F.Cu at (132.5, 41.5)
- added REF**: MountingHole_3.2mm_M3, MountingHole:MountingHole_3.2mm_M3, F.Cu at (132.5, 134.5)
- added REF**: PinSocket_1x05_P2.54mm_Vertical, Connector_PinSocket_2.54mm:PinSocket_1x05_P2.54mm_Vertical, B.Cu at (129.0, 116.5)
- added REF**: PinSocket_1x05_P2.54mm_Vertical, Connector_PinSocket_2.54mm:PinSocket_1x05_P2.54mm_Vertical, B.Cu at (110.0, 97.5)
- added REF**: PinSocket_1x05_P2.54mm_Vertical, Connector_PinSocket_2.54mm:PinSocket_1x05_P2.54mm_Vertical, B.Cu at (129.0, 59.5)
- added REF**: PinSocket_1x05_P2.54mm_Vertical, Connector_PinSocket_2.54mm:PinSocket_1x05_P2.54mm_Vertical, B.Cu at (53.0, 59.5)
- added REF**: PinSocket_1x05_P2.54mm_Vertical, Connector_PinSocket_2.54mm:PinSocket_1x05_P2.54mm_Vertical, B.Cu at (91.0, 78.5)
- C19, C20, R13, R16, R17, R18: moved to B.Cu
- CB5: moved to F.Cu
- moved U2 514.2 mm to (568.5, 91.5)
- moved R17 412.1 mm to (133.5, 52.1), turned to -90 degrees
- moved J2 406.8 mm to (474.0, 182.3)
- moved L1 406.8 mm to (449.0, 186.0)
- moved U1 406.8 mm to (463.0, 180.2)
- moved U3 406.8 mm to (483.2, 174.0)
- moved Y1 350.9 mm to (377.4, 141.6)
- moved SW1 348.3 mm to (366.5, 145.9)
- moved J1 348.3 mm to (374.8, 131.6)
- moved LEDB4 325.6 mm to (354.5, 144.0), turned to 0 degrees
- moved LEDB3 318.3 mm to (354.4, 137.6), turned to 0 degrees
- moved LEDB5 310.0 mm to (354.3, 155.2)
- moved CB1 304.6 mm to (376.0, 190.5)
- moved CB3 304.6 mm to (386.5, 190.5)
- moved CB2 304.6 mm to (380.9, 190.5)
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Connections:
- R5 pad 1: USBDM -> USBDP
Routing:
- net Vusb: track 17.1 -> 501.7 mm, vias 0 -> 16
- net COL5: track 86.6 -> 110.9 mm
- net Net-(C19-Pad1): track 0.00 -> 21.3 mm
- net GND: track 0.00 -> 19.2 mm, vias 0 -> 2
- net Net-(LED55-Pad2): track 0.00 -> 15.6 mm
- net COL4: track 85.5 -> 99.8 mm, vias 4 -> 5
- net ROTD: track 82.6 -> 95.4 mm
- net ROTA: track 0.00 -> 12.7 mm
- net COL3: track 85.6 -> 97.5 mm, vias 4 -> 5
- net ROW2: track 81.5 -> 91.4 mm
- net ROW3: track 81.5 -> 90.3 mm
- net ROW4: track 81.5 -> 89.3 mm
- net ROW5: track 81.5 -> 89.3 mm
- net COL1: track 94.6 -> 101.8 mm
- net COL2: track 85.6 -> 92.7 mm, vias 4 -> 5
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- added copper zone on B.Cu, net GND
- added copper zone on F.Cu, net Vusb

Commit message: Added board interconnectors
And started redoing the board interconnects -- the previous solution
lacked symmetry and elegance (= looked like a dog's breakfast).
Parts:
- removed the REF** at (52.5, 116.5)
- removed the REF** at (129.0, 116.5)
- removed the REF** at (110.0, 97.5)
- removed the REF** at (129.0, 59.5)
- removed the REF** at (53.0, 59.5)
- removed the REF** at (91.0, 78.5)
- added J3: Conn_01x08_Male, Connector_PinSocket_2.54mm:PinSocket_1x08_P2.54mm_Vertical, F.Cu at (114.0, 195.0)
- added J4: Conn_01x08_Male, Connector_PinSocket_2.54mm:PinSocket_1x08_P2.54mm_Vertical, B.Cu at (38.0, 79.1)
- added J5: Conn_01x08_Female, Connector_PinSocket_2.54mm:PinSocket_1x08_P2.54mm_Vertical, B.Cu at (77.3, 135.0)
- added J6: Conn_01x08_Female, Connector_PinSocket_2.54mm:PinSocket_1x08_P2.54mm_Vertical, F.Cu at (100.7, 195.0)
Connections:
- net BACKLIGHT renamed BACKLIGHTIN
- net Net-(LED55-Pad2) renamed BACKLIGHTOUT
- R13 pad 1: Net-(C19-Pad1) -> ROTB
- R13 pad 2: ROTB -> Net-(C19-Pad1)
Routing:
- net Vusb: track 501.7 -> 399.7 mm, vias 16 -> 13
- net ROTD: track 95.4 -> 39.2 mm
- net Net-(LED41-Pad2): track 28.0 -> 0.00 mm
- net Net-(LED21-Pad2): track 27.1 -> 0.00 mm
- net ROW5: track 89.3 -> 112.8 mm
- net Net-(C19-Pad1): track 21.3 -> 2.78 mm
- net GND: track 19.2 -> 1.05 mm, vias 2 -> 0
- net BACKLIGHTOUT: track 15.6 -> 0.00 mm
- net ROTA: track 12.7 -> 0.00 mm
- net COL5: track 110.9 -> 98.7 mm
- net COL4: track 99.8 -> 87.6 mm
- net ROW2: track 91.4 -> 103.0 mm
- net COL3: track 97.5 -> 87.8 mm
- net COL1: track 101.8 -> 94.6 mm
- net ROW4: track 89.3 -> 95.4 mm
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
Commit message: Redid board connectors, started 2nd board
Parts:
- added ?: , , F.Cu at (240.0, 38.0)
- added ?: , , F.Cu at (240.0, 138.0)
- added ?: , , F.Cu at (140.0, 38.0)
- added ?: , , F.Cu at (140.0, 138.0)
- added J10: Conn_01x03_Female, Connector_PinSocket_2.54mm:PinSocket_1x03_P2.54mm_Vertical, F.Cu at (142.0, 66.5)
- added J11: Conn_01x03_Male, Connector_PinSocket_2.54mm:PinSocket_1x03_P2.54mm_Vertical, B.Cu at (102.4, 136.0)
- added J12: Conn_01x03_Male, Connector_PinSocket_2.54mm:PinSocket_1x03_P2.54mm_Vertical, B.Cu at (64.5, 136.0)
- added J13: Conn_01x03_Female, Connector_PinSocket_2.54mm:PinSocket_1x03_P2.54mm_Vertical, F.Cu at (206.5, 136.0)
- added J14: Conn_01x03_Female, Connector_PinSocket_2.54mm:PinSocket_1x03_P2.54mm_Vertical, F.Cu at (168.5, 136.0)
- added J15: Conn_01x03_Male, Connector_PinSocket_2.54mm:PinSocket_1x03_P2.54mm_Vertical, B.Cu at (134.0, 66.5)
- added J16: Conn_01x03_Female, Connector_PinSocket_2.54mm:PinSocket_1x03_P2.54mm_Vertical, F.Cu at (238.0, 66.5)
- added J7: Conn_01x03_Male, Connector_PinSocket_2.54mm:PinSocket_1x03_P2.54mm_Vertical, B.Cu at (38.0, 104.5)
- added J8: Conn_01x03_Male, Connector_PinSocket_2.54mm:PinSocket_1x03_P2.54mm_Vertical, B.Cu at (38.0, 66.5)
- added J9: Conn_01x03_Female, Connector_PinSocket_2.54mm:PinSocket_1x03_P2.54mm_Vertical, F.Cu at (142.0, 104.5)
- J3: value Conn_01x08_Male -> Conn_01x03_Male; footprint Connector_PinSocket_2.54mm:PinSocket_1x08_P2.54mm_Vertical -> Connector_PinSocket_2.54mm:PinSocket_1x03_P2.54mm_Vertical; moved to B.Cu
- J4: value Conn_01x08_Male -> Conn_01x03_Male; footprint Connector_PinSocket_2.54mm:PinSocket_1x08_P2.54mm_Vertical -> Connector_PinSocket_2.54mm:PinSocket_1x03_P2.54mm_Vertical
- J5: value Conn_01x08_Female -> Conn_01x03_Female; footprint Connector_PinSocket_2.54mm:PinSocket_1x08_P2.54mm_Vertical -> Connector_PinSocket_2.54mm:PinSocket_1x03_P2.54mm_Vertical; moved to F.Cu
- J6: value Conn_01x08_Female -> Conn_01x03_Female; footprint Connector_PinSocket_2.54mm:PinSocket_1x08_P2.54mm_Vertical -> Connector_PinSocket_2.54mm:PinSocket_1x03_P2.54mm_Vertical
- LEDB1, LEDB2, LEDB3, LEDB4, LEDB5, LEDB6, LEDB7, LEDB8, R13, R16, R17, R18: moved to F.Cu
- R14: moved to B.Cu
- moved R14 380.5 mm to (42.5, 55.0), turned to 90 degrees
- moved R5 380.5 mm to (186.5, 50.0), turned to 180 degrees
- moved U2 378.5 mm to (190.0, 90.0), turned to 135 degrees
- moved C3 373.9 mm to (183.2, 86.8), turned to 45 degrees
- moved R4 365.0 mm to (193.0, 48.0), turned to 180 degrees
- moved D2 341.8 mm to (238.0, 97.0), turned to 180 degrees
- moved C_R2 339.5 mm to (235.2, 104.9), turned to 90 degrees
- moved R3 324.4 mm to (193.3, 103.0)
- moved D3 323.8 mm to (238.0, 95.0), turned to 180 degrees
- moved J2 316.5 mm to (190.0, 42.6)
- moved U1 301.6 mm to (190.0, 52.0)
- moved U3 294.4 mm to (208.5, 68.2)
- moved C4 277.5 mm to (186.8, 96.8), turned to 135 degrees
- moved R12 275.1 mm to (234.8, 95.0), turned to 180 degrees
- moved C_R3 266.6 mm to (200.6, 79.6), turned to 135 degrees
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Connections:
- J3 pad 2: BACKLIGHTOUT -> GND
- J3 pad 3: COL1 -> Vusb
- J4 pad 2: BACKLIGHTIN -> Vusb
- J4 pad 3: ROTD -> Vusb
- J5 pad 2: BACKLIGHTOUT -> GND
- J5 pad 3: COL1 -> Vusb
- J6 pad 2: BACKLIGHTIN -> Vusb
- J6 pad 3: ROTD -> Vusb
Routing:
- net Vusb: track 399.7 -> 107.0 mm, vias 13 -> 25
- net ROTD: track 39.2 -> 104.9 mm
- net COL3: track 87.8 -> 116.7 mm
- net BACKLIGHTOUT: track 0.00 -> 26.6 mm, vias 0 -> 1
- net Net-(LED41-Pad2): track 0.00 -> 23.4 mm, vias 0 -> 2
- net Net-(LED21-Pad2): track 0.00 -> 23.0 mm, vias 0 -> 2
- net Net-(C19-Pad1): track 2.78 -> 24.5 mm
- net Net-(C17-Pad2): track 0.00 -> 17.9 mm
- net ROW5: track 112.8 -> 96.4 mm
- net ROW3: track 85.7 -> 101.5 mm
- net COL1: track 94.6 -> 110.0 mm
- net ROW2: track 103.0 -> 87.7 mm
- net COL2: track 87.7 -> 102.8 mm
- net COL4: track 87.6 -> 102.7 mm
- net BACKLIGHTIN: track 0.00 -> 14.8 mm, vias 0 -> 1
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Other:
- board size 100 x 100 mm -> 204 x 100 mm

Commit message: Adjusted to 4 layer board
- USB interface is most important, lets route that first.

- leds interconnect will mess with everybody, so push those to the
  internal layer.

- do away with quirky 45 degree placing
Parts:
- C1, C2, C3, C4, C5: moved to B.Cu
- moved C1 314.3 mm to (180.3, 85.2), turned to 180 degrees
- moved C16 311.8 mm to (148.2, 56.5), turned to -90 degrees
- moved R1 308.4 mm to (198.2, 45.0), turned to 90 degrees
- moved L1 285.5 mm to (177.7, 97.2), turned to 135 degrees
- moved C9 273.7 mm to (164.0, 56.5), turned to 90 degrees
- moved C7 271.8 mm to (180.4, 93.9), turned to -45 degrees
- moved CB4 262.8 mm to (158.0, 71.8), turned to -135 degrees
- moved CB5 261.5 mm to (173.8, 56.2), turned to -135 degrees
- moved C_R1 255.0 mm to (232.0, 110.2), turned to 90 degrees
- moved CB3 244.1 mm to (158.0, 104.5), turned to -45 degrees
- moved R15 228.5 mm to (219.6, 110.6), turned to 45 degrees
- moved R7 222.6 mm to (187.8, 80.3), turned to 90 degrees
- moved CB2 219.1 mm to (173.5, 120.0), turned to -45 degrees
- moved C8 215.2 mm to (161.8, 56.5), turned to 90 degrees
- moved C6 214.6 mm to (179.0, 95.5), turned to -45 degrees
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Connections:
- net Net-(R7-Pad1) renamed /USBD+
- net Net-(R8-Pad1) renamed /USBD-
- net USBDM renamed USBDN
- C6 pad 1: unconnected-(C6-Pad1) -> Net-(C6-Pad1)
- C7 pad 1: unconnected-(C7-Pad1) -> Net-(C6-Pad1)
- C7 pad 2: unconnected-(C7-Pad2) -> GND
- L1 pad 2: Net-(L1-Pad2) -> Net-(C6-Pad1)
- U2 pad 9: Net-(L1-Pad2) -> Net-(C6-Pad1)
Routing:
- net Vusb: track 107.0 -> 162.2 mm, vias 25 -> 29
- net COL1: track 110.0 -> 153.3 mm, vias 5 -> 6
- net COL2: track 102.8 -> 143.3 mm, vias 5 -> 6
- net USBDP: track 5.96 -> 44.0 mm
- net COL3: track 116.7 -> 154.1 mm, vias 5 -> 6
- net Net-(LEDB7-Pad2): track 0.00 -> 36.1 mm, vias 0 -> 2
- net Net-(LEDB3-Pad2): track 0.00 -> 36.1 mm, vias 0 -> 2
- net Net-(LEDB1-Pad2): track 0.00 -> 35.9 mm, vias 0 -> 2
- net Net-(LEDB5-Pad2): track 0.00 -> 35.9 mm, vias 0 -> 2
- net USBDN: track 5.96 -> 40.8 mm, vias 0 -> 2
- net Net-(LEDB6-Pad2): track 0.00 -> 17.9 mm, vias 0 -> 2
- net Net-(LEDB4-Pad2): track 0.00 -> 17.9 mm, vias 0 -> 2
- net Net-(LEDB2-Pad2): track 0.00 -> 17.9 mm, vias 0 -> 2
- net BACKLIGHTOUT: track 26.6 -> 41.2 mm
- net Net-(C17-Pad2): track 17.9 -> 9.75 mm
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- added copper zone on B.Cu, net +3V3
- added copper zone on F.Cu, net GND
- added copper zone on B.Cu, net Vusb
Other:
- copper layers 2 -> 4
- board text added: "Keyboard switch board uses only 2 layers"
- board text added: "MCU board 4 layers"
